File: AntennaPCB.brd (EAGLE design)
At the start: 43.2 x 38.1 mm, 28 parts, among them Q1 27.12MHz

Commit message: Created the antenna board and adjusted sizing of the board
Parts:
- removed J1: (no value), BM02B-ACHSS-GAN-TF_LF__SN_:JST_BM02B-ACHSS-GAN-TF(LF)(SN)
- removed R7: 0, Resistor_Capacitor:RES_1206
- removed U$2: T2I-02, SeniorDesignParts:T2I-02
Connections:
- removed net ANTC_1: J1.1, R5.1, U$2.P$1
- removed net ANTC_2: J1.2, R6.1, U$2.P$2
- removed net N$7: J1.S1, J1.S2, R7.1
- new net ANTENNA: R5.1, R6.1
- net GND: no longer R7.2
Routing:
- net ANTENNA: track 0.00 -> 546.6 mm, vias 0 -> 3
- net N$7: track 18.4 -> 0.00 mm
- net ANTC_2: track 10.6 -> 0.00 mm
- net ANTC_1: track 10.6 -> 0.00 mm
Other:
- board size 43.2 x 38.1 mm -> 76.2 x 38.1 mm

Commit message: Moved more stuff around and edited via sizes
Routing:
- net GND: vias 2 -> 9
Other:
- board text added: "Antenna Board V1 Group 15 Dabble Melchor De La Garza Cynthia Zatlokowicz"
Changed lines of the file:
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@@
 <wire x1="76.2" y1="38.1" x2="0" y2="38.1" width="0" layer="20"/>
 <wire x1="0" y1="38.1" x2="0" y2="0" width="0" layer="20"/>
+<text x="28" y="0.4" size="1" layer="125">Antenna Board V1
+Group 15 Dabble
+Melchor De La Garza
+Cynthia Zatlokowicz</text>
 </plain>
 <attributes>
@@
 <wire x1="21.5392" y1="2.7432" x2="25.1206" y2="6.3246" width="0.254" layer="1"/>
 <wire x1="25.1206" y1="6.3246" x2="25.1206" y2="14.263" width="0.254" layer="1"/>
+<via x="23.8" y="8.2" extent="1-16" drill="0.35"/>
+<via x="24.7" y="2.1" extent="1-16" drill="0.35"/>
+<via x="15.3" y="8.2" extent="1-16" drill="0.35"/>
+<via x="2.3" y="7.4" extent="1-16" drill="0.35"/>
+<via x="24" y="22.6" extent="1-16" drill="0.35"/>
+<via x="3" y="22.3" extent="1-16" drill="0.35"/>
+<via x="19.7" y="11.2" extent="1-16" drill="0.35"/>
 </signal>
 <signal name="SCLK">
@@
 <wire x1="52.501821875" y1="17.9198" x2="51.765221875" y2="17.1832" width="0.2032" layer="16"/>
 </signal>
-<signal name="N$4">
-<via x="19.7" y="11.2" extent="1-16" drill="0.35"/>
-</signal>
-<signal name="N$8">
-<via x="2.3" y="7.4" extent="1-16" drill="0.35"/>
-</signal>
-<signal name="N$12">
-<via x="3" y="22.3" extent="1-16" drill="0.35"/>
-</signal>
-<signal name="N$13">
-<via x="15.3" y="8.2" extent="1-16" drill="0.35"/>
-</signal>
-<signal name="N$14">
-<via x="24" y="22.6" extent="1-16" drill="0.35"/>
-</signal>
-<signal name="N$15">
-<via x="22.7" y="9.3" extent="1-16" drill="0.35"/>
-</signal>
-<signal name="N$16">
-<via x="24.7" y="2.1" extent="1-16" drill="0.35"/>
-</signal>
 </signals>
 <mfgpreviewcolors>
@@
 </drawing>
 <compatibility>
+<note version="6.3" minversion="6.2.2" severity="warning">
+Since Version 6.2.2 text objects can contain more than one line,
+which will not be processed correctly with this version.
+</note>
 <note version="8.2" severity="warning">
 Since Version 8.2, EAGLE supports online libraries. The ids

Commit message: Put stand-offs on the board
Parts:
- added H1, H2, H3: STAND-OFF, SparkFun-Hardware:STAND-OFF
Changed lines of the file:
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@@
 <wire x1="76.2" y1="38.1" x2="0" y2="38.1" width="0" layer="20"/>
 <wire x1="0" y1="38.1" x2="0" y2="0" width="0" layer="20"/>
-<text x="28" y="0.4" size="1" layer="125">Antenna Board V1
+<text x="17.5" y="31.6" size="1" layer="125">Antenna Board V1
 Group 15 Dabble
 Melchor De La Garza
@@
 </element>
 <element name="U$1" library="SeniorDesignParts" package="HVQFN32" value="MFRC522" x="12.6812" y="13.7404" rot="R90"/>
+<element name="H1" library="SparkFun-Hardware" library_urn="urn:adsk.eagle:library:519" package="STAND-OFF" package3d_urn="urn:adsk.eagle:package:38630/1" value="STAND-OFF" x="40" y="34"/>
+<element name="H2" library="SparkFun-Hardware" library_urn="urn:adsk.eagle:library:519" package="STAND-OFF" package3d_urn="urn:adsk.eagle:package:38630/1" value="STAND-OFF" x="40" y="3.2"/>
+<element name="H3" library="SparkFun-Hardware" library_urn="urn:adsk.eagle:library:519" package="STAND-OFF" package3d_urn="urn:adsk.eagle:package:38630/1" value="STAND-OFF" x="2.9" y="27"/>
 </elements>
 <signals>
